File: carrier_board_ESP32/carrier_board_ESP32.kicad_sch (KiCad schematic)
At the start: 68 parts, among them IC1 A3144, IC2 A3144, IC3 SS49E, IC4 SS49E, IC5 SS49E, IC6 SS49E, IC7 SS49E, IC8 SS49E, J1 Conn_01x02_Socket, J12 LTR390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

Commit message: cleaning repo
Parts:
- added D3: D, Diode_SMD:D_SMA, symbol Device:D
Connections:
- net 5V_supply: now also U3.4 (EN), D3.1 (K)
- net BATT+: now also D3.2 (A)
- net GND: no longer U3.4 (EN)
Changed lines of the file:
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@@
 	)
 	(junction
+		(at 64.77 21.59)
+		(diameter 0)
+		(color 0 0 0 0)
+	)
+	(junction
 		(at 26.67 137.16)
 		(diameter 0)
@@
 	)
 	(junction
+		(at 39.37 118.11)
+		(diameter 0)
+		(color 0 0 0 0)
+	)
+	(junction
 		(at 19.05 49.53)
 		(diameter 0)
@@
 	)
 	(junction
+		(at 92.71 57.15)
+		(diameter 0)
+		(color 0 0 0 0)
+	)
+	(junction
 		(at 85.09 138.43)
 		(diameter 0)
@@
 	(wire
 		(pts
-			(xy 39.37 128.27) (xy 39.37 139.7)
-		)
-		(stroke
-			(width 0)
-			(type default)
-		)
-	)
-	(wire
-		(pts
 			(xy 46.99 160.02) (xy 49.53 160.02)
 		)
@@
 	(wire
 		(pts
+			(xy 92.71 21.59) (xy 64.77 21.59)
+		)
+		(stroke
+			(width 0)
+			(type default)
+		)
+	)
+	(wire
+		(pts
 			(xy 87.63 90.17) (xy 87.63 91.44)
 		)
@@
 	(wire
 		(pts
+			(xy 92.71 45.72) (xy 92.71 21.59)
+		)
+		(stroke
+			(width 0)
+			(type default)
+		)
+	)
+	(wire
+		(pts
 			(xy 201.93 58.42) (xy 208.28 58.42)
 		)
@@
 	(wire
 		(pts
+			(xy 39.37 118.11) (xy 39.37 128.27)
+		)
+		(stroke
+			(width 0)
+			(type default)
+		)
+	)
+	(wire
+		(pts
 			(xy 69.85 118.11) (xy 74.93 118.11)
 		)
@@
 	(wire
 		(pts
-			(xy 33.02 118.11) (xy 41.91 118.11)
+			(xy 33.02 118.11) (xy 39.37 118.11)
 		)
 		(stroke
@@
 	(wire
 		(pts
+			(xy 92.71 53.34) (xy 92.71 57.15)
+		)
+		(stroke
+			(width 0)
+			(type default)
+		)
+	)
+	(wire
+		(pts
 			(xy 85.09 118.11) (xy 85.09 125.73)
 		)
@@
 	(wire
 		(pts
+			(xy 64.77 21.59) (xy 64.77 22.86)
+		)
+		(stroke
+			(width 0)
+			(type default)
+		)
+	)
+	(wire
+		(pts
 			(xy 64.77 30.48) (xy 64.77 41.91)
 		)
@@
 	(wire
 		(pts
-			(xy 80.01 57.15) (xy 93.98 57.15)
+			(xy 80.01 57.15) (xy 92.71 57.15)
 		)
 		(stroke
@@
 	(wire
 		(pts
-			(xy 64.77 20.32) (xy 64.77 22.86)
+			(xy 64.77 17.78) (xy 64.77 21.59)
 		)
 		(stroke
@@
 	(wire
 		(pts
+			(xy 92.71 57.15) (xy 93.98 57.15)
+		)
+		(stroke
+			(width 0)
+			(type default)
+		)
+	)
+	(wire
+		(pts
 			(xy 186.69 158.75) (xy 191.77 158.75)
 		)
@@
 	(wire
 		(pts
+			(xy 39.37 118.11) (xy 41.91 118.11)
+		)
+		(stroke
+			(width 0)
+			(type default)
+		)
+	)
+	(wire
+		(pts
 			(xy 134.62 142.24) (xy 139.7 142.24)
 		)
@@
 	)
 	(label "5V_supply"
-		(at 64.77 20.32 0)
+		(at 64.77 17.78 0)
 		(effects
 			(font
@@
 	)
 	(symbol
-		(lib_id "power:GND")
-		(at 39.37 139.7 0)
-		(unit 1)
-		(exclude_from_sim no)
-		(in_bom yes)
-		(on_board yes)
-		(dnp no)
-		(fields_autoplaced yes)
-		(property "Reference" "#PWR119"
-			(at 39.37 146.05 0)
-			(effects
-				(font
-					(size 1.27 1.27)
-				)
-				(hide yes)
-			)
-		)
-		(property "Value" "GND"
-			(at 39.37 144.78 0)
-			(effects
-				(font
-					(size 1.27 1.27)
-				)
-			)
-		)
-		(property "Footprint" ""
-			(at 39.37 139.7 0)
-			(effects
-				(font
-					(size 1.27 1.27)
-				)
-				(hide yes)
-			)
-		)
-		(property "Datasheet" ""
-			(at 39.37 139.7 0)
-			(effects
-				(font
-					(size 1.27 1.27)
-				)
-				(hide yes)
-			)
-		)
-		(property "Description" "Power symbol creates a global label with name \"GND\" , ground"
-			(at 39.37 139.7 0)
-			(effects
-				(font
-					(size 1.27 1.27)
-				)
-				(hide yes)
-			)
-		)
-		(pin "1"
-		)
-		(instances
-			(project "carrier_board_ESP32"
-				(path "/3cb3161a-672b-452c-99c3-9aad76a0c868"
-					(reference "#PWR119")
-					(unit 1)
-				)
-			)
-		)
-	)
-	(symbol
 		(lib_id "Device:R_Small")
 		(at 66.04 121.92 0)
@@
 					(unit 1)
 				)
+			)
+		)
+	)
+	(symbol
+		(lib_id "Device:D")
+		(at 92.71 49.53 270)
+		(unit 1)
+		(exclude_from_sim no)
+		(in_bom yes)
+		(on_board yes)
+		(dnp no)
+		(fields_autoplaced yes)
+		(property "Reference" "D3"
+			(at 95.25 48.2599 90)
+			(effects
+				(font
+					(size 1.27 1.27)
+				)
+				(justify left)
+			)
+		)
+		(property "Value" "D"
+			(at 95.25 50.7999 90)
+			(effects
+				(font
+					(size 1.27 1.27)
+				)
+				(justify left)
+			)
+		)
+		(property "Footprint" "Diode_SMD:D_SMA"
+			(at 92.71 49.53 0)
+			(effects
+				(font
+					(size 1.27 1.27)
+				)
+				(hide yes)
+			)
+		)
+		(property "Datasheet" "~"
+			(at 92.71 49.53 0)
+			(effects
+				(font
+					(size 1.27 1.27)
+				)
+				(hide yes)
+			)
+		)
+		(property "Description" "Diode"
+			(at 92.71 49.53 0)
+			(effects
+				(font
+					(size 1.27 1.27)
+				)
+				(hide yes)
+			)
+		)
+		(property "Sim.Device" "D"
+			(at 92.71 49.53 0)
+			(effects
+				(font
+					(size 1.27 1.27)
+				)
+				(hide yes)
+			)
+		)
+		(property "Sim.Pins" "1=K 2=A"
+			(at 92.71 49.53 0)
+			(effects
+				(font
+					(size 1.27 1.27)
+				)
+				(hide yes)
+			)
+		)
+		(pin "2"
+		)
+		(pin "1"
+		)
+		(instances
+			(project ""
+				(path "/3cb3161a-672b-452c-99c3-9aad76a0c868"
+					(reference "D3")
+					(unit 1)
+				)
